File: BitBadge.kicad_pcb (KiCad board)
At the start: 2 copper layers, 64 x 67.1 mm, 72 parts, among them SW1 SW_2P3T

Commit message: new handouts and kicad8
Connections:
- SW1 pad 2: Net-(SW1-Pad2) -> unconnected-(SW1A-B-Pad2)
- SW1 pad 6: Net-(SW1-Pad6) -> unconnected-(SW1-Pad6)
Other:
- net class Default removed
